Commit message: Changed Urdf limits and pid values

File: urdf/manipulator.urdf (robot description, URDF)
Before this commit: robot manipulator, 5 links, 4 joints
Links:
- added link world
Joints:
- added joint dummy_joint: type fixed, parent world, child link_0
- joint joint_1: limit lower=0.0 upper=3.14159265359 effort=0.0 velocity=0.0 -> lower=0.0 upper=3.14159265359 effort=1.0 velocity=1.0
- joint joint_2: limit lower=0.0 upper=3.14159265359 effort=0.0 velocity=0.0 -> lower=0.0 upper=3.14159265359 effort=1.0 velocity=0.0
- joint joint_3: limit lower=0.0 upper=3.14159265359 effort=0.0 velocity=0.0 -> lower=0.0 upper=3.14159265359 effort=1.0 velocity=0.0
